File: kicad/usb_co2_7seg.kicad_pcb (KiCad board)
At the start: 2 copper layers, 95 x 72 mm, 16 parts, among them U1 PinHeader_XIAO, U2 PinHeader_XIAO, U3 SeeeduinoXIAO, U4 MH-Z19B, U5 TM1637, U6 7segment_led, U7 SW_push_2pin

Commit message: 配線済み DRC ok
Routing:
- net +5V: track 0.00 -> 123.8 mm
- net Net-(D1-Pad2): track 0.00 -> 111.1 mm, vias 0 -> 1
- net Net-(R1-Pad2): track 0.00 -> 108.8 mm, vias 0 -> 2
- net Net-(U5-Pad4): track 0.00 -> 91.0 mm
- net Net-(U5-Pad3): track 0.00 -> 90.3 mm, vias 0 -> 1
- net Net-(U5-Pad5): track 0.00 -> 83.9 mm
- net Net-(U5-Pad7): track 0.00 -> 79.9 mm
- net Net-(U5-Pad2): track 0.00 -> 73.6 mm
- net Net-(U5-Pad9): track 0.00 -> 64.9 mm
- net Net-(R3-Pad2): track 0.00 -> 63.5 mm
- net Net-(R4-Pad2): track 0.00 -> 62.9 mm
- net Net-(U5-Pad8): track 0.00 -> 60.1 mm
- net Net-(U5-Pad14): track 0.00 -> 59.6 mm
- net Net-(U5-Pad13): track 0.00 -> 59.6 mm
- net Net-(U5-Pad15): track 0.00 -> 57.5 mm
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- added copper zone on B.Cu, net GND
- added copper zone on F.Cu, net GND
